File: es-board/digital.kicad_sch (KiCad schematic)
At the start: 30 parts, among them J1 DNP, J2 Conn_01x04, Q5 IRF530NSTRLPB, SW1 SW_SPST, SW2 SW_SPST, SW3 SW_SPST, SW4 SW_SPST, SW5 SW_SPST, U2 ATmega32U4-A, U5 OLED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

Commit message: Design review tweaks
Other:
- note added: "TODO fix direction"
- moved on the sheet: R15, R16, TP3
Changed lines of the file:
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@@
     (stroke (width 0) (type default))
   )
-  (wire (pts (xy 119.38 91.44) (xy 113.03 91.44))
+  (wire (pts (xy 119.38 91.44) (xy 112.395 91.44))
     (stroke (width 0) (type default))
   )
@@
     (stroke (width 0) (type default))
   )
-  (wire (pts (xy 119.38 88.9) (xy 113.03 88.9))
+  (wire (pts (xy 119.38 88.9) (xy 112.395 88.9))
     (stroke (width 0) (type default))
   )
@@
     (stroke (width 0) (type default))
   )
-  (wire (pts (xy 105.41 88.9) (xy 100.33 88.9))
+  (wire (pts (xy 104.775 88.9) (xy 100.33 88.9))
     (stroke (width 0) (type default))
   )
@@
     (stroke (width 0) (type default))
   )
-  (wire (pts (xy 100.33 93.98) (xy 111.76 93.98))
+  (wire (pts (xy 100.33 93.98) (xy 110.49 93.98))
     (stroke (width 0) (type default))
   )
@@
     (stroke (width 0) (type default))
   )
-  (wire (pts (xy 105.41 91.44) (xy 100.33 91.44))
+  (wire (pts (xy 104.775 91.44) (xy 100.33 91.44))
     (stroke (width 0) (type default))
   )
@@
     (stroke (width 0) (type default))
   )
-  (polyline (pts (xy 129.54 99.06) (xy 190.5 99.06))
+  (polyline (pts (xy 137.16 99.06) (xy 198.12 99.06))
     (stroke (width 0.5) (type default) (color 192 0 0 1))
   )
@@
     (stroke (width 0) (type default))
   )
-  (wire (pts (xy 100.33 96.52) (xy 111.76 96.52))
+  (wire (pts (xy 100.33 96.52) (xy 110.49 96.52))
     (stroke (width 0) (type default))
   )
@@
   )
   (text "a5" (at 90.17 120.65 0)
+    (effects (font (size 1.27 1.27)) (justify left bottom))
+  )
+  (text "TODO fix direction" (at 146.05 102.235 0)
     (effects (font (size 1.27 1.27)) (justify left bottom))
   )
@@
     )
   )
-  (symbol (lib_id "Graphic:SYM_Arrow_Large") (at 194.31 99.06 0) (unit 1)
+  (symbol (lib_id "Graphic:SYM_Arrow_Large") (at 133.35 99.06 180) (unit 1)
     (in_bom no) (on_board no) (dnp no) (fields_autoplaced)
-    (property "Reference" "#SYM1" (at 194.31 96.774 0)
-      (effects (font (size 1.27 1.27)) hide)
-    )
-    (property "Value" "SYM_Arrow_Large" (at 194.31 101.092 0)
-      (effects (font (size 1.27 1.27)) hide)
-    )
-    (property "Footprint" "" (at 194.31 99.06 0)
-      (effects (font (size 1.27 1.27)) hide)
-    )
-    (property "Datasheet" "~" (at 194.31 99.06 0)
-      (effects (font (size 1.27 1.27)) hide)
-    )
-    (property "Sim.Enable" "0" (at 194.31 99.06 0)
+    (property "Reference" "#SYM1" (at 133.35 101.346 0)
+      (effects (font (size 1.27 1.27)) hide)
+    )
+    (property "Value" "SYM_Arrow_Large" (at 133.35 97.028 0)
+      (effects (font (size 1.27 1.27)) hide)
+    )
+    (property "Footprint" "" (at 133.35 99.06 0)
+      (effects (font (size 1.27 1.27)) hide)
+    )
+    (property "Datasheet" "~" (at 133.35 99.06 0)
+      (effects (font (size 1.27 1.27)) hide)
+    )
+    (property "Sim.Enable" "0" (at 133.35 99.06 0)
       (effects (font (size 1.27 1.27)) hide)
     )
@@
     )
   )
-  (symbol (lib_id "Device:R") (at 109.22 91.44 90) (unit 1)
+  (symbol (lib_id "Device:R") (at 108.585 91.44 90) (unit 1)
     (in_bom yes) (on_board yes) (dnp no)
-    (property "Reference" "R16" (at 104.14 90.17 90)
-      (effects (font (size 1.27 1.27)))
-    )
-    (property "Value" "0" (at 109.22 91.44 90)
-      (effects (font (size 1.27 1.27)))
-    )
-    (property "Footprint" "Resistor_SMD:R_1206_3216Metric" (at 109.22 93.218 90)
-      (effects (font (size 1.27 1.27)) hide)
-    )
-    (property "Datasheet" "~" (at 109.22 91.44 0)
+    (property "Reference" "R16" (at 103.505 90.17 90)
+      (effects (font (size 1.27 1.27)))
+    )
+    (property "Value" "0" (at 108.585 91.44 90)
+      (effects (font (size 1.27 1.27)))
+    )
+    (property "Footprint" "Resistor_SMD:R_1206_3216Metric" (at 108.585 93.218 90)
+      (effects (font (size 1.27 1.27)) hide)
+    )
+    (property "Datasheet" "~" (at 108.585 91.44 0)
       (effects (font (size 1.27 1.27)) hide)
     )
@@
     )
   )
-  (symbol (lib_id "Connector_Generic:Conn_01x02") (at 116.84 93.98 0) (unit 1)
-    (in_bom yes) (on_board yes) (dnp no) (fields_autoplaced)
-    (property "Reference" "TP3" (at 118.872 94.0379 0)
-      (effects (font (size 1.27 1.27)) (justify left))
-    )
-    (property "Value" "Conn_01x02" (at 118.872 96.4621 0)
-      (effects (font (size 1.27 1.27)) (justify left))
-    )
-    (property "Footprint" "Connector_PinHeader_2.54mm:PinHeader_1x02_P2.54mm_Vertical" (at 116.84 93.98 0)
-      (effects (font (size 1.27 1.27)) hide)
-    )
-    (property "Datasheet" "~" (at 116.84 93.98 0)
+  (symbol (lib_id "Connector_Generic:Conn_01x02") (at 115.57 93.98 0) (unit 1)
+    (in_bom yes) (on_board yes) (dnp no) (fields_autoplaced)
+    (property "Reference" "TP3" (at 117.602 94.0379 0)
+      (effects (font (size 1.27 1.27)) (justify left))
+    )
+    (property "Value" "Conn_01x02" (at 117.602 96.4621 0)
+      (effects (font (size 1.27 1.27)) (justify left))
+    )
+    (property "Footprint" "Connector_PinHeader_2.54mm:PinHeader_1x02_P2.54mm_Vertical" (at 115.57 93.98 0)
+      (effects (font (size 1.27 1.27)) hide)
+    )
+    (property "Datasheet" "~" (at 115.57 93.98 0)
       (effects (font (size 1.27 1.27)) hide)
     )
@@
     )
   )
-  (symbol (lib_id "Device:R") (at 109.22 88.9 90) (unit 1)
+  (symbol (lib_id "Device:R") (at 108.585 88.9 90) (unit 1)
     (in_bom yes) (on_board yes) (dnp no)
-    (property "Reference" "R15" (at 104.14 87.63 90)
-      (effects (font (size 1.27 1.27)))
-    )
-    (property "Value" "0" (at 109.22 88.9 90)
-      (effects (font (size 1.27 1.27)))
-    )
-    (property "Footprint" "Resistor_SMD:R_1206_3216Metric" (at 109.22 90.678 90)
-      (effects (font (size 1.27 1.27)) hide)
-    )
-    (property "Datasheet" "~" (at 109.22 88.9 0)
-      (effects (font (size 1.27 1.27)) hide)
-    )
+    (property "Reference" "R15" (at 103.505 87.63 90)
+      (effects (font (size 1.27 1.27)))
+    )
+    (property "Value" "0" (at 108.585 88.9 90)
+      (effects (font (size 1.27 1.27)))
+    )
+    (property "Footprint" "Resistor_SMD:R_1206_3216Metric" (at 108.585 90.678 90)
+      (effects (font (size 1.27 1.27)) hide)
+    )
+    (property "Datasheet" "~" (at 108.585 88.9 0)
+      (effects (font (size 1.27 1.27)) hide)
+    )

Commit message: updated BOM
Parts:
- J2: value Conn_01x04 -> DNP
- R15, R16: DPN (none) -> RMCF1206ZT0R00CT-ND; MPN (none) -> RMCF1206ZT0R00
- TP1, TP2: value TestPoint -> DNP
- TP3: value Conn_01x02 -> DNP
- U2: MPN IC MCU 8BIT 32KB FLASH 44TQFP -> ATMEGA32U4-AUR
Changed lines of the file:
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@@
   (title_block
     (title "ExploSnake")
-    (date "2023-10-19")
-    (rev "r1")
+    (date "2023-11-15")
+    (rev "r1.0")
     (company "Team 2")
   )
@@
       (effects (font (size 1.27 1.27)) (justify left))
     )
-    (property "Value" "Conn_01x04" (at 238.252 47.0479 0)
+    (property "Value" "DNP" (at 238.252 47.0479 0)
       (effects (font (size 1.27 1.27)) (justify left))
     )
@@
       (effects (font (size 1.27 1.27)) (justify left))
     )
-    (property "Value" "TestPoint" (at 105.537 99.5101 0)
+    (property "Value" "DNP" (at 105.537 99.5101 0)
       (effects (font (size 1.27 1.27)) (justify left))
     )
@@
       (effects (font (size 1.27 1.27)) hide)
     )
+    (property "DPN" "RMCF1206ZT0R00CT-ND" (at 108.585 91.44 0)
+      (effects (font (size 1.27 1.27)) hide)
+    )
+    (property "MPN" "RMCF1206ZT0R00" (at 108.585 91.44 0)
+      (effects (font (size 1.27 1.27)) hide)
+    )
     (pin "1")
     (pin "2")
@@
       (effects (font (size 1.27 1.27)) (justify left))
     )
-    (property "Value" "TestPoint" (at 105.537 56.3301 0)
+    (property "Value" "DNP" (at 105.537 56.3301 0)
       (effects (font (size 1.27 1.27)) (justify left))
     )
@@
       (effects (font (size 1.27 1.27)) hide)
     )
-    (property "MPN" "IC MCU 8BIT 32KB FLASH 44TQFP" (at 85.09 96.52 0)
+    (property "MPN" "ATMEGA32U4-AUR" (at 85.09 96.52 0)
       (effects (font (size 1.27 1.27)) hide)
     )
@@
       (effects (font (size 1.27 1.27)) (justify left))
     )
-    (property "Value" "Conn_01x02" (at 117.602 96.4621 0)
+    (property "Value" "DNP" (at 117.602 96.4621 0)
       (effects (font (size 1.27 1.27)) (justify left))
     )
@@
       (effects (font (size 1.27 1.27)) hide)
     )
+    (property "DPN" "RMCF1206ZT0R00CT-ND" (at 108.585 88.9 0)
+      (effects (font (size 1.27 1.27)) hide)
+    )
+    (property "MPN" "RMCF1206ZT0R00" (at 108.585 88.9 0)
+      (effects (font (size 1.27 1.27)) hide)
+    )
