File: es-board/es-board.kicad_pcb (KiCad board)
At the start: 2 copper layers, 77.9 x 44.5 mm, 63 parts, among them J1 DNP, J2 Conn_01x04, J3 USB_C_Receptacle_USB2.0, Q1 Q_PMOS_GSD, Q2 Q_PMOS_GSD, Q3 Q_PMOS_GSD, Q4 Q_PMOS_GSD, Q5 IRF530NSTRLPB, SW1 SW_SPST, SW2 SW_SPST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

Commit message: Added test plan
Parts:
- J2: value Conn_01x04 -> DNP
- TP1, TP2: value TestPoint -> DNP
- TP3: value Conn_01x02 -> DNP
Connections:
- U1 pad 10: unconnected-(U1-FLIP-Pad10) -> FLIP
Changed lines of the file:
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@@
   (net 37 "unconnected-(U1-HPI_INT-Pad7)")
   (net 38 "unconnected-(U1-GPIO_1-Pad8)")
-  (net 39 "unconnected-(U1-FLIP-Pad10)")
+  (net 39 "FLIP")
   (net 40 "unconnected-(U1-HPI_SDA-Pad12)")
   (net 41 "unconnected-(U1-HPI_SCL-Pad13)")
@@
       (net 15 "USB_PD_FAULT") (pinfunction "FAULT") (pintype "input"))
     (pad "10" smd roundrect (at 0.25 -1.9875 90) (size 0.25 0.775) (layers "B.Cu" "B.Paste" "B.Mask") (roundrect_rratio 0.25)
-      (net 39 "unconnected-(U1-FLIP-Pad10)") (pinfunction "FLIP") (pintype "input+no_connect"))
+      (net 39 "FLIP") (pinfunction "FLIP") (pintype "input"))
     (pad "11" smd roundrect (at 0.75 -1.9875 90) (size 0.25 0.775) (layers "B.Cu" "B.Paste" "B.Mask") (roundrect_rratio 0.25)
       (net 9 "VBUS") (pinfunction "VDC_OUT") (pintype "input"))
@@
     (tags "capacitor")
     (property "DPN" "1276-6736-1-ND")
-    (property "MPN" "CAP CER 10UF 50V X5R 1206")
+    (property "MPN" "CL31A106MBHNNNE")
     (property "Sheetfile" "power.kicad_sch")
     (property "Sheetname" "Power")
@@
     (descr "Resistor SMD 1206 (3216 Metric), square (rectangular) end terminal, IPC_7351 nominal, (Body size source: IPC-SM-782 page 72, https://www.pcb-3d.com/wordpress/wp-content/uploads/ipc-sm-782a_amendment_1_and_2.pdf), generated with kicad-footprint-generator")
     (tags "resistor")
+    (property "DPN" "RMCF1206ZT0R00CT-ND")
+    (property "MPN" "RMCF1206ZT0R00")
     (property "Sheetfile" "digital.kicad_sch")
     (property "Sheetname" "Digital")
@@
     (tags "capacitor")
     (property "DPN" "1276-6736-1-ND")
-    (property "MPN" "CAP CER 10UF 50V X5R 1206")
+    (property "MPN" "CL31A106MBHNNNE")
     (property "Sheetfile" "power.kicad_sch")
     (property "Sheetname" "Power")
@@
     (descr "Resistor SMD 1206 (3216 Metric), square (rectangular) end terminal, IPC_7351 nominal, (Body size source: IPC-SM-782 page 72, https://www.pcb-3d.com/wordpress/wp-content/uploads/ipc-sm-782a_amendment_1_and_2.pdf), generated with kicad-footprint-generator")
     (tags "resistor")
+    (property "DPN" "RMCF1206ZT0R00CT-ND")
+    (property "MPN" "RMCF1206ZT0R00")
     (property "Sheetfile" "digital.kicad_sch")
     (property "Sheetname" "Digital")
@@
         (effects (font (size 0.8 0.8) (thickness 0.12)) (justify mirror))
     )
-    (fp_text value "Conn_01x02" (at 0 -4.87) (layer "B.Fab")
+    (fp_text value "DNP" (at 0 -4.87) (layer "B.Fab")
         (effects (font (size 1 1) (thickness 0.15)) (justify mirror))
     )
@@
     (tags "QFP 0.8")
     (property "DPN" "ATMEGA32U4-AURCT-ND")
-    (property "MPN" "IC MCU 8BIT 32KB FLASH 44TQFP")
+    (property "MPN" "ATMEGA32U4-AUR")
     (property "Sheetfile" "digital.kicad_sch")
     (property "Sheetname" "Digital")
@@
         (effects (font (size 0.8 0.8) (thickness 0.12)) (justify mirror))
     )
-    (fp_text value "TestPoint" (at 0 -1.56) (layer "B.Fab")
+    (fp_text value "DNP" (at 0 -1.56) (layer "B.Fab")
         (effects (font (size 1 1) (thickness 0.15)) (justify mirror))
     )
@@
         (effects (font (size 0.8 0.8) (thickness 0.12)) (justify mirror))
     )
-    (fp_text value "Conn_01x04" (at 0 -9.95 90) (layer "B.Fab")
+    (fp_text value "DNP" (at 0 -9.95 90) (layer "B.Fab")
         (effects (font (size 1 1) (thickness 0.15)) (justify mirror))
     )
@@
         (effects (font (size 0.8 0.8) (thickness 0.12)) (justify mirror))
     )
-    (fp_text value "TestPoint" (at 0 -1.56) (layer "B.Fab")
+    (fp_text value "DNP" (at 0 -1.56) (layer "B.Fab")
         (effects (font (size 1 1) (thickness 0.15)) (justify mirror))
     )
